File: arisutea-pcb.kicad_pcb (KiCad board)
At the start: 2 copper layers, 339.1 x 121 mm, 182 parts, among them J12 VCC, J13 D+, J14 D-, J15 GND, J16 RGB, J17 RGB TO J18, J18 RGB FROM J17, J2 MISO, J3 +5V, J4 SCK, J5 MOSI, J6 ~RES~, J7 GND, SW1 SW_Push, SW10 SW_Push, SW11 SW_Push, SW12 SW_Push, SW13 SW_Push, SW14 SW_Push, SW15 SW_Push, SW16 SW_Push, SW17 SW_Push, SW18 SW_Push, SW19 SW_Push, SW2 SW_Push, SW20 SW_Push, SW21 SW_Push, SW22 SW_Push, SW23 SW_Push, SW24 SW_Push, SW25 SW_Push, SW26 SW_Push, SW27 SW_Push, SW28 SW_Push, SW29 SW_Push, SW3 SW_Push, SW30 SW_Push, SW31 SW_Push, SW32 SW_Push, SW33 SW_Push, SW34 SW_Push, SW35 SW_Push, SW36 SW_Push, SW37 SW_Push, SW38 SW_Push, SW39 SW_Push, SW4 SW_Push, SW40 SW_Push, SW41 SW_Push, SW42 SW_Push, SW43 SW_Push, SW44 SW_Push, SW45 SW_Push, SW46 SW_Push, SW47 SW_Push, SW48 SW_Push, SW49 SW_Push, SW5 SW_Push, SW50 SW_Push, SW51 SW_Push, SW52 SW_Push, SW53 SW_Push, SW54 SW_Push, SW55 SW_Push, SW56 SW_Push, SW57 SW_Push, SW58 SW_Push, SW59 SW_Push, SW6 SW_Push, SW60 SW_Push, SW61 SW_Push, SW62 SW_Push, SW63 SW_Push, SW64 SW_Push, SW65 SW_Push, SW66 SW_Push, SW7 SW_Push, SW8 SW_Push, SW9 SW_Push, U1 USBLC6-2SC6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

Commit message: initial STM32 design
Parts:
- removed J12: VCC, arisutea:PinHeader_1x01_P2.54mm_Vertical
- removed J13: D+, arisutea:PinHeader_1x01_P2.54mm_Vertical
- removed J14: D-, arisutea:PinHeader_1x01_P2.54mm_Vertical
- removed J15, J7: GND, arisutea:PinHeader_1x01_P2.54mm_Vertical
- removed J16: RGB, arisutea:PinHeader_1x03_P2.54mm_Vertical
- removed J17: RGB TO J18, arisutea:PinHeader_1x03_P2.54mm_Vertical
- removed J18: RGB FROM J17, arisutea:PinHeader_1x03_P2.54mm_Vertical
- removed J2: MISO, arisutea:PinHeader_1x01_P2.54mm_Vertical
- removed J3: +5V, arisutea:PinHeader_1x01_P2.54mm_Vertical
- removed J4: SCK, arisutea:PinHeader_1x01_P2.54mm_Vertical
- removed J5: MOSI, arisutea:PinHeader_1x01_P2.54mm_Vertical
- removed J6: ~RES~, arisutea:PinHeader_1x01_P2.54mm_Vertical
- removed R5, R6: 5k1, arisutea:R_0805_2012Metric_Pad1.20x1.40mm_HandSolder
- removed Y1: Crystal_GND24, arisutea:Crystal_SMD_TXC_7M-4Pin_3.2x2.5mm_HandSoldering
- added C10: 1u, 3x6_components:C_0805_2012Metric_Pad1.18x1.45mm_HandSolder, B.Cu at (170.2, 35.0)
- added C11: 100n, 3x6_components:C_0805_2012Metric_Pad1.18x1.45mm_HandSolder, B.Cu at (179.5, 104.4)
- added C12: 100n, 3x6_components:C_0805_2012Metric_Pad1.18x1.45mm_HandSolder, B.Cu at (173.9, 104.1)
- added D67: SMF6.0CA, 3x6_components:D_SOD-123, B.Cu at (164.5, 28.4)
- added J1: Conn_Generic_Conn_01x08, 3x6_connectors:PinHeader_2x04_P2.54mm_Vertical, F.Cu at (166.2, 100.7)
- added LOGO3: arm_logo, 3x6_graphics:ARM_powered, B.Cu at (71.6, 118.1)
- added LOGO4: arm_logo, 3x6_graphics:ARM_powered, F.Cu at (71.8, 118.1)
- added LOGO5: qmk_logo, 3x6_graphics:QMK_Logo_Light, B.Cu at (286.8, 108.4)
- added LOGO6: qmk_logo, 3x6_graphics:QMK_Logo_Light, F.Cu at (286.5, 108.5)
- added Q1: 2N7002, 3x6_components:SOT-23, B.Cu at (179.5, 109.0)
- added R10: 470, 3x6_components:R_0805_2012Metric_Pad1.20x1.40mm_HandSolder, B.Cu at (135.8, 27.7)
- added R11: 470, 3x6_components:R_0805_2012Metric_Pad1.20x1.40mm_HandSolder, B.Cu at (130.3, 27.7)
- added U3: NUF2221W1T2G, 3x6_components:SOT-23-6_Handsoldering, B.Cu at (175.5, 37.8)
- C1: value 22pF -> 10n; footprint arisutea:C_0805_2012Metric_Pad1.18x1.45mm_HandSolder -> 3x6_components:C_0805_2012Metric_Pad1.18x1.45mm_HandSolder
- C2: value 22pF -> 100n; footprint arisutea:C_0805_2012Metric_Pad1.18x1.45mm_HandSolder -> 3x6_components:C_0805_2012Metric_Pad1.18x1.45mm_HandSolder
- C3: value 10uF -> 100n; footprint arisutea:C_0805_2012Metric_Pad1.18x1.45mm_HandSolder -> 3x6_components:C_0805_2012Metric_Pad1.18x1.45mm_HandSolder
- C4: value 1uF (±10%) -> 1u; footprint arisutea:C_0805_2012Metric_Pad1.18x1.45mm_HandSolder -> 3x6_components:C_0805_2012Metric_Pad1.18x1.45mm_HandSolder
- C5: value 1uF -> 100n; footprint arisutea:C_0805_2012Metric_Pad1.18x1.45mm_HandSolder -> 3x6_components:C_0805_2012Metric_Pad1.18x1.45mm_HandSolder
- C6, C8: value 0.1uF -> 4.7u; footprint arisutea:C_0805_2012Metric_Pad1.18x1.45mm_HandSolder -> 3x6_components:C_0805_2012Metric_Pad1.18x1.45mm_HandSolder
- C7: value 0.1uF -> 4.7n; footprint arisutea:C_0805_2012Metric_Pad1.18x1.45mm_HandSolder -> 3x6_components:C_0805_2012Metric_Pad1.18x1.45mm_HandSolder
- C9: value 0.1uF -> 1u; footprint arisutea:C_0805_2012Metric_Pad1.18x1.45mm_HandSolder -> 3x6_components:C_0805_2012Metric_Pad1.18x1.45mm_HandSolder
- F1: footprint arisutea:Fuse_1206_3216Metric_Pad1.42x1.75mm_HandSolder -> 3x6_components:Fuse_1206_3216Metric_Pad1.42x1.75mm_HandSolder
- H1, H2, H3, H4, H5, H6, H7, H8: footprint arisutea:Plated_Through_Hole_M2 -> 3x6_mounting_hole:Plated_Through_Hole_M2
- LED1: value NUM_LOCK -> LED; footprint arisutea:LED_IN-S124ARUW -> 3x6_components:LED_IN-S124ARUW
- LED2: value CAPS_LOCK -> LED; footprint arisutea:LED_IN-S124ARUW -> 3x6_components:LED_IN-S124ARUW
- LED3: value FN_LED -> LED; footprint arisutea:LED_IN-S124ARUW -> 3x6_components:LED_IN-S124ARUW
- R1: value 22 -> 1M; footprint arisutea:R_0805_2012Metric_Pad1.20x1.40mm_HandSolder -> 3x6_components:R_0805_2012Metric_Pad1.20x1.40mm_HandSolder
- R2: value 22 -> 5k1; footprint arisutea:R_0805_2012Metric_Pad1.20x1.40mm_HandSolder -> 3x6_components:R_0805_2012Metric_Pad1.20x1.40mm_HandSolder
- R3: value 10K -> 5k1; footprint arisutea:R_0805_2012Metric_Pad1.20x1.40mm_HandSolder -> 3x6_components:R_0805_2012Metric_Pad1.20x1.40mm_HandSolder
- R4, R9: footprint arisutea:R_0805_2012Metric_Pad1.20x1.40mm_HandSolder -> 3x6_components:R_0805_2012Metric_Pad1.20x1.40mm_HandSolder
- R7, R8: value 470 -> 10K; footprint arisutea:R_0805_2012Metric_Pad1.20x1.40mm_HandSolder -> 3x6_components:R_0805_2012Metric_Pad1.20x1.40mm_HandSolder
- SWR1: footprint arisutea:SW_SPST_TL3342 -> 3x6_components:SW_SPST_TL3342
- U1: value USBLC6-2SC6 -> STM32F072-LQFP48; footprint arisutea:SOT-23-6_Handsoldering -> 3x6_components:LQFP-48_7x7mm_P0.5mm
- U2: value ATmega32U4-AU -> TLV70233; footprint arisutea:TQFP-44_10x10mm_P0.8mm -> 3x6_components:SOT-23-5_HandSoldering
- USB1: footprint arisutea:USB_C_Receptacle_HRO_TYPE-C-31-M-12-HandSoldering -> 3x6_components:USB_C_Receptacle_HRO_TYPE-C-31-M-12-HandSoldering
- moved R7 87.5 mm to (179.5, 106.4), turned to 0 degrees
- moved R8 87.2 mm to (173.9, 106.1), turned to 0 degrees
- moved SWR1 84.6 mm to (186.1, 112.4)
- moved C4 73.2 mm to (173.9, 102.2), turned to 0 degrees
- moved U1 61.1 mm to (170.3, 91.9), turned to 135 degrees
- moved C1 60.0 mm to (173.9, 100.2), turned to 0 degrees
- moved C2 59.4 mm to (160.8, 92.5), turned to 180 degrees
- moved C5 54.7 mm to (179.1, 90.2)
- moved C3 54.0 mm to (172.8, 82.2)
- moved R4 51.2 mm to (179.5, 102.5), turned to 180 degrees
- moved C8 45.0 mm to (160.8, 90.5), turned to 180 degrees
- moved C6 43.0 mm to (170.9, 82.2), turned to 270 degrees
- moved C9 27.6 mm to (161.6, 35.0), turned to 270 degrees
- moved R1 25.3 mm to (184.9, 34.6), turned to 270 degrees
- moved R3 22.4 mm to (171.2, 31.6), turned to 0 degrees
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Connections:
- C1 pad 1: GND -> +3V3
- C1 pad 2: XTAL1 -> GND
- C2 pad 1: XTAL2 -> +3V3
- C3 pad 1: +5V -> +3V3
- C4 pad 1: Net-(C4-Pad1) -> +3V3
- C5 pad 1: +5V -> +3V3
- C6 pad 1: +5V -> GND
- C6 pad 2: GND -> +3V3
- C7 pad 1: +5V -> Net-(C7-Pad1)
- C8 pad 1: +5V -> +3V3
- C9 pad 1: +5V -> VBUS
- D1 pad 1: /row0 -> row0
- D10 pad 1: /row0 -> row0
- D11 pad 1: /row1 -> row1
- D12 pad 1: /row2 -> row2
- D13 pad 1: /row3 -> row3
- D14 pad 1: /row4 -> row4
- D15 pad 1: /row0 -> row0
- D16 pad 1: /row1 -> row1
- D17 pad 1: /row2 -> row2
- D18 pad 1: /row3 -> row3
- D19 pad 1: /row0 -> row0
- D2 pad 1: /row1 -> row1
- D20 pad 1: /row1 -> row1
- D21 pad 1: /row2 -> row2
- D22 pad 1: /row3 -> row3
- D23 pad 1: /row4 -> row4
- D24 pad 1: /row0 -> row0
- D25 pad 1: /row1 -> row1
- D26 pad 1: /row2 -> row2
- D27 pad 1: /row3 -> row3
- D28 pad 1: /row4 -> row4
- D29 pad 1: /row0 -> row0
- D3 pad 1: /row2 -> row2
- D30 pad 1: /row1 -> row1
- D31 pad 1: /row2 -> row2
- D32 pad 1: /row3 -> row3
- D33 pad 1: /row0 -> row0
- D34 pad 1: /row1 -> row1
- D35 pad 1: /row2 -> row2
- D36 pad 1: /row3 -> row3
- D37 pad 1: /row4 -> row4
- D38 pad 1: /row0 -> row0
- D39 pad 1: /row1 -> row1
- D4 pad 1: /row3 -> row3
- D40 pad 1: /row2 -> row2
- D41 pad 1: /row3 -> row3
- D42 pad 1: /row0 -> row0
- D43 pad 1: /row1 -> row1
- D44 pad 1: /row2 -> row2
- D45 pad 1: /row3 -> row3
- D46 pad 1: /row4 -> row4
- D47 pad 1: /row0 -> row0
- D48 pad 1: /row1 -> row1
- D49 pad 1: /row2 -> row2
- D5 pad 1: /row4 -> row4
- D50 pad 1: /row3 -> row3
- D51 pad 1: /row0 -> row0
- D52 pad 1: /row1 -> row1
- D53 pad 1: /row2 -> row2
- D54 pad 1: /row3 -> row3
- D55 pad 1: /row0 -> row0
- D56 pad 1: /row1 -> row1
- D57 pad 1: /row2 -> row2
- D58 pad 1: /row4 -> row4
- D59 pad 1: /row0 -> row0
- D6 pad 1: /row0 -> row0
- D60 pad 1: /row1 -> row1
- D61 pad 1: /row3 -> row3
- D62 pad 1: /row4 -> row4
- D63 pad 1: /row1 -> row1
- D64 pad 1: /row2 -> row2
- D65 pad 1: /row3 -> row3
- D66 pad 1: /row4 -> row4
- D7 pad 1: /row1 -> row1
- D8 pad 1: /row2 -> row2
- D9 pad 1: /row3 -> row3
- F1 pad 1: +5V -> VBUS
- F1 pad 2: VCC -> Net-(F1-Pad2)
- LED1 pad C: GND -> led1
- LED2 pad C: GND -> led2
- LED3 pad C: GND -> led3
- R1 pad 1: D+ -> Net-(C7-Pad1)
- R1 pad 2: Net-(J13-Pad1) -> GND
- R2 pad 1: D- -> Net-(R2-Pad1)
- R2 pad 2: Net-(J14-Pad1) -> GND
- R3 pad 1: +5V -> GND
- R3 pad 2: /~RES~ -> Net-(R3-Pad2)
- R4 pad 1: Net-(R4-Pad1) -> boot0
- R7 pad 1: Net-(LED1-PadA) -> Net-(C11-Pad2)
- R7 pad 2: FN_L -> GND
- R8 pad 1: Net-(LED2-PadA) -> +3V3
- R8 pad 2: CAPS_L -> NRST
- R9 pad 1: Net-(LED3-PadA) -> VBUS
- R9 pad 2: NUM_L -> Net-(LED1-PadA)
- SW1 pad 2: /col0 -> col0
- SW10 pad 2: /col2 -> col2
- SW11 pad 2: /col2 -> col2
- SW12 pad 2: /col2 -> col2
- SW13 pad 2: /col2 -> col2
- SW14 pad 2: /col2 -> col2
- SW15 pad 2: /col3 -> col3
- SW16 pad 2: /col3 -> col3
- SW17 pad 2: /col3 -> col3
- SW18 pad 2: /col3 -> col3
- SW19 pad 2: /col4 -> col4
- SW2 pad 2: /col0 -> col0
- SW20 pad 2: /col4 -> col4
- SW21 pad 2: /col4 -> col4
- SW22 pad 2: /col4 -> col4
- SW23 pad 2: /col4 -> col4
- SW24 pad 2: /col5 -> col5
- SW25 pad 2: /col5 -> col5
- SW26 pad 2: /col5 -> col5
- SW27 pad 2: /col5 -> col5
- SW28 pad 2: /col5 -> col5
- SW29 pad 2: /col6 -> col6
- SW3 pad 2: /col0 -> col0
- SW30 pad 2: /col6 -> col6
- SW31 pad 2: /col6 -> col6
- SW32 pad 2: /col6 -> col6
- SW33 pad 2: /SCK -> col7
- SW34 pad 2: /SCK -> col7
- SW35 pad 2: /SCK -> col7
- SW36 pad 2: /SCK -> col7
- SW37 pad 2: /SCK -> col7
- SW38 pad 2: /col8 -> col8
- SW39 pad 2: /col8 -> col8
- SW4 pad 2: /col0 -> col0
- SW40 pad 2: /col8 -> col8
- SW41 pad 2: /col8 -> col8
- SW42 pad 2: /col9 -> col9
- SW43 pad 2: /col9 -> col9
- SW44 pad 2: /col9 -> col9
- SW45 pad 2: /col9 -> col9
- SW46 pad 2: /col9 -> col9
- SW47 pad 2: /col10 -> col10
- SW48 pad 2: /col10 -> col10
- SW49 pad 2: /col10 -> col10
- SW5 pad 2: /col0 -> col0
- SW50 pad 2: /col10 -> col10
- SW51 pad 2: /col11 -> col11
- SW52 pad 2: /col11 -> col11
- SW53 pad 2: /col11 -> col11
- SW54 pad 2: /col11 -> col11
- SW55 pad 2: /col12 -> col12
- SW56 pad 2: /col12 -> col12
- SW57 pad 2: /col12 -> col12
- SW58 pad 2: /col12 -> col12
- SW59 pad 2: /col13 -> col13
- SW6 pad 2: /col1 -> col1
- SW60 pad 2: /col13 -> col13
- SW61 pad 2: /col13 -> col13
- SW62 pad 2: /col13 -> col13
- SW63 pad 2: /MISO -> col14
- SW64 pad 2: /MISO -> col14
- SW65 pad 2: /MISO -> col14
- SW66 pad 2: /MISO -> col14
- SW7 pad 2: /col1 -> col1
- SW8 pad 2: /col1 -> col1
- SW9 pad 2: /col1 -> col1
- SWR1 pad 1: GND -> boot0
- SWR1 pad 2: /~RES~ -> +3V3
- U1 pad 1: Net-(U1-Pad1) -> +3V3
- U1 pad 2: GND -> row2
- U1 pad 3: Net-(U1-Pad3) -> row3
- U1 pad 4: Net-(J13-Pad1) -> row4
- U1 pad 5: VCC -> Net-(U1-Pad5)
- U1 pad 6: Net-(J14-Pad1) -> Net-(U1-Pad6)
- U2 pad 1: /col2 -> VBUS
- U2 pad 2: +5V -> GND
- U2 pad 3: D- -> VBUS
- U2 pad 4: D+ -> Net-(U2-Pad4)
- U2 pad 5: GND -> +3V3
- USB1 pad A4: VCC -> Net-(F1-Pad2)
- USB1 pad A5: Net-(R5-Pad1) -> Net-(R3-Pad2)
- USB1 pad A6: Net-(U1-Pad3) -> Net-(U3-Pad6)
- USB1 pad A7: Net-(U1-Pad1) -> Net-(U3-Pad4)
- USB1 pad A9: VCC -> Net-(F1-Pad2)
- USB1 pad B5: Net-(R6-Pad1) -> Net-(R2-Pad1)
- USB1 pad B6: Net-(U1-Pad3) -> Net-(U3-Pad6)
- USB1 pad B7: Net-(U1-Pad1) -> Net-(U3-Pad4)
- USB1 pad S1: GND -> Net-(C7-Pad1)
Routing:
- net GND: track 677.1 -> 226.2 mm, vias 20 -> 18
- net /row3: track 442.5 -> 0.00 mm, vias 2 -> 0
- net /row4: track 434.3 -> 0.00 mm, vias 2 -> 0
- net /row2: track 406.1 -> 0.00 mm, vias 2 -> 0
- net /row1: track 388.9 -> 0.00 mm, vias 4 -> 0
- net row3: track 0.00 -> 380.9 mm
- net row4: track 0.00 -> 378.3 mm, vias 0 -> 2
- net row1: track 0.00 -> 342.1 mm, vias 0 -> 2
- net row2: track 0.00 -> 340.0 mm, vias 0 -> 2
- net /row0: track 324.2 -> 0.00 mm, vias 4 -> 0
- net row0: track 0.00 -> 313.7 mm, vias 0 -> 2
- net +5V: track 312.4 -> 0.00 mm, vias 7 -> 0
- net /col12: track 298.9 -> 0.00 mm, vias 5 -> 0
- net /col13: track 297.6 -> 0.00 mm, vias 5 -> 0
- net col14: track 0.00 -> 295.9 mm, vias 0 -> 4
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Other:
- board text added: "Arisutea STM32 v0.1 3x6 Design mattyams"
- board text removed: "+5V"
- board text removed: "Arisutea Rev 0.6 3x6 Design mattyams"
- board text removed: "DATA"
- board text removed: "GND"

Commit message: routing and placement work
Parts:
- added C13: 100n, 3x6_components:C_0805_2012Metric_Pad1.18x1.45mm_HandSolder, B.Cu at (173.9, 104.1)
- C1: value 10n -> 100n
- C11, C3: value 100n -> 1u
- C2: value 100n -> 10n
- C4: value 1u -> 100n
- C5: value 100n -> 4.7u
- C6, C8: value 4.7u -> 100n
- C7: value 4.7n -> 4.7u
- C9: value 1u -> 4.7n
- moved C11 70.0 mm to (170.2, 35.0), turned to 90 degrees
- moved C7 49.0 mm to (172.7, 82.5), turned to 315 degrees
- moved C9 21.3 mm to (182.9, 34.6)
- moved C3 20.0 mm to (173.9, 102.2), turned to 180 degrees
- moved C8 18.3 mm to (179.1, 90.2), turned to 0 degrees
- moved C5 18.1 mm to (161.4, 94.0), turned to 45 degrees
- moved C2 15.2 mm to (173.9, 100.2)
- moved C4 13.0 mm to (162.8, 95.4), turned to 45 degrees
- moved C1 9.55 mm to (179.1, 92.2)
- moved C10 8.51 mm to (161.7, 35.0), turned to 270 degrees
- moved C12 5.53 mm to (179.5, 104.4)
- moved C6 1.78 mm to (171.2, 83.9), turned to 315 degrees
- moved Q1 0.06 mm to (179.5, 109.0)
- turned D67 to 90 degrees
Connections:
- C1 pad 1: +3V3 -> GND
- C1 pad 2: GND -> 3.3V
- C10 pad 1: +3V3 -> 5V
- C11 pad 1: boot0 -> 3.3V
- C11 pad 2: Net-(C11-Pad2) -> GND
- C12 pad 1: NRST -> boot0
- C12 pad 2: GND -> Net-(C12-Pad2)
- C2 pad 1: +3V3 -> GND
- C2 pad 2: GND -> 3.3V
- C3 pad 1: +3V3 -> GND
- C3 pad 2: GND -> 3.3V
- C4 pad 1: +3V3 -> GND
- C4 pad 2: GND -> 3.3V
- C5 pad 1: +3V3 -> GND
- C5 pad 2: GND -> 3.3V
- C6 pad 2: +3V3 -> 3.3V
- C7 pad 1: Net-(C7-Pad1) -> GND
- C7 pad 2: GND -> 3.3V
- C8 pad 1: +3V3 -> GND
- C8 pad 2: GND -> 3.3V
- C9 pad 1: VBUS -> Net-(C9-Pad1)
- D63 pad 1: row1 -> row0
- D64 pad 1: row2 -> row1
- D65 pad 1: row3 -> row2
- D67 pad 1: GND -> 5V
- D67 pad 2: VBUS -> GND
- F1 pad 1: VBUS -> 5V
- J1 pad 8: +3V3 -> 3.3V
- Q1 pad 1: Net-(C11-Pad2) -> Net-(C12-Pad2)
- R1 pad 1: Net-(C7-Pad1) -> Net-(C9-Pad1)
- R10 pad 1: VBUS -> 5V
- R11 pad 1: VBUS -> 5V
- R7 pad 1: Net-(C11-Pad2) -> Net-(C12-Pad2)
- R8 pad 1: +3V3 -> 3.3V
- R9 pad 1: VBUS -> 5V
- SWR1 pad 2: +3V3 -> 3.3V
- U1 pad 1: +3V3 -> 3.3V
- U1 pad 24: +3V3 -> 3.3V
- U1 pad 36: +3V3 -> 3.3V
- U1 pad 48: +3V3 -> 3.3V
- U1 pad 9: +3V3 -> 3.3V
- U2 pad 1: VBUS -> 5V
- U2 pad 3: VBUS -> 5V
- U2 pad 5: +3V3 -> 3.3V
- U3 pad 5: +3V3 -> 3.3V
- USB1 pad S1: Net-(C7-Pad1) -> Net-(C9-Pad1)
Routing:
- net 3.3V: track 0.00 -> 191.9 mm, vias 0 -> 6
- net +3V3: track 182.2 -> 0.00 mm, vias 6 -> 0
- net VBUS: track 64.6 -> 0.00 mm, vias 2 -> 0
- net 5V: track 0.00 -> 56.7 mm, vias 0 -> 2
- net row3: track 380.9 -> 336.8 mm
- net row0: track 313.7 -> 344.5 mm
- net Net-(C9-Pad1): track 0.00 -> 26.4 mm
- net Net-(C7-Pad1): track 26.4 -> 0.00 mm
- net row1: track 342.1 -> 331.8 mm
- net GND: track 226.2 -> 218.2 mm, vias 18 -> 16
- net row2: track 340.0 -> 333.3 mm
- net col14: track 295.9 -> 289.3 mm
- net col4: track 118.0 -> 123.6 mm
- net col13: track 268.1 -> 271.8 mm
- net Net-(C12-Pad2): track 0.00 -> 3.70 mm
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
Commit message: big update
Re-routed everything. Moved components around. Corrected gerbers and BOM/POS.  Updated library. Added renders.
Parts:
- C1, C10, C11, C12, C13, C2, C3, C4, C5, C6, C7, C8, C9: footprint 3x6_components:C_0805_2012Metric_Pad1.18x1.45mm_HandSolder -> arisutea:C_0805_2012Metric_Pad1.18x1.45mm_HandSolder
- D67: footprint 3x6_components:D_SOD-123 -> arisutea:D_SOD-123
- F1: footprint 3x6_components:Fuse_1206_3216Metric_Pad1.42x1.75mm_HandSolder -> arisutea:Fuse_1206_3216Metric_Pad1.42x1.75mm_HandSolder
- H1, H2, H3, H4, H5, H6, H7, H8: footprint 3x6_mounting_hole:Plated_Through_Hole_M2 -> arisutea:Generic-Mounthole
- J1: footprint 3x6_connectors:PinHeader_2x04_P2.54mm_Vertical -> arisutea:PinHeader_2x04_P2.54mm_Vertical
- LED1, LED2, LED3: footprint 3x6_components:LED_IN-S124ARUW -> arisutea:LED_IN-S124ARUW
- LOGO3, LOGO4: footprint 3x6_graphics:ARM_powered -> arisutea:Logo_ARM_powered
- LOGO5, LOGO6: footprint 3x6_graphics:QMK_Logo_Light -> arisutea:Logo_QMK_Light
- Q1: footprint 3x6_components:SOT-23 -> arisutea:SOT-23
- R1, R10, R11, R2, R3, R4, R7, R8, R9: footprint 3x6_components:R_0805_2012Metric_Pad1.20x1.40mm_HandSolder -> arisutea:R_0805_2012Metric_Pad1.20x1.40mm_HandSolder
- SWR1: footprint 3x6_components:SW_SPST_TL3342 -> arisutea:SW_SPST_TL3342
- U1: footprint 3x6_components:LQFP-48_7x7mm_P0.5mm -> arisutea:LQFP-48_7x7mm_P0.5mm
- U2: footprint 3x6_components:SOT-23-5_HandSoldering -> arisutea:SOT-23-5_HandSoldering
- U3: footprint 3x6_components:SOT-23-6_Handsoldering -> arisutea:SOT-363_SC-70-6_Handsoldering
- USB1: footprint 3x6_components:USB_C_Receptacle_HRO_TYPE-C-31-M-12-HandSoldering -> arisutea:USB_C_Receptacle_HRO_TYPE-C-31-M-12-HandSoldering
- moved SWR1 8.41 mm to (177.8, 113.9), turned to 0 degrees
- moved C3 4.32 mm to (173.3, 97.9), turned to 225 degrees
- moved C13 3.96 mm to (175.4, 107.8)
- moved R8 3.96 mm to (175.4, 109.8)
- moved C1 3.31 mm to (178.9, 88.9), turned to 135 degrees
- moved C5 2.17 mm to (162.7, 95.8), turned to 135 degrees
- moved C8 1.72 mm to (177.4, 90.3), turned to 135 degrees
- moved C4 1.62 mm to (164.1, 94.4), turned to 135 degrees
- moved C6 1.53 mm to (170.1, 84.9)
- moved C7 1.53 mm to (171.5, 83.5)
- moved C2 1.20 mm to (174.7, 99.3), turned to 225 degrees
Connections:
- U1 pad 10: Net-(U1-Pad10) -> (no net)
- U1 pad 11: Net-(U1-Pad11) -> (no net)
- U1 pad 18: Net-(U1-Pad18) -> (no net)
- U1 pad 19: Net-(U1-Pad19) -> (no net)
- U1 pad 5: Net-(U1-Pad5) -> (no net)
- U1 pad 6: Net-(U1-Pad6) -> (no net)
- U2 pad 4: Net-(U2-Pad4) -> (no net)
- USB1 pad A8: Net-(USB1-PadA8) -> (no net)
- USB1 pad B8: Net-(USB1-PadB8) -> (no net)
Routing:
- net 3.3V: track 191.9 -> 169.0 mm, vias 6 -> 5
- net row3: track 336.8 -> 328.0 mm
- net row4: track 378.4 -> 369.7 mm
- net GND: track 218.2 -> 209.7 mm, vias 16 -> 15
- net boot0: track 31.8 -> 37.2 mm
- net col11: track 210.5 -> 208.1 mm
- net Net-(F1-Pad2): track 15.7 -> 17.4 mm
- net row1: track 331.8 -> 331.0 mm
- net NRST: track 20.6 -> 20.1 mm
Other:
- net class Power: trace_width 0.381 -> 0.6
- board text added: "3.3V"
- board text added: "Arisutea STM32 v0.2 3x6 Design mattyams"
- board text added: "CS"
- board text added: "GND"
- board text added: "IRQ"
- board text added: "MOSI"
- board text added: "RES"
- board text added: "SCK"
- board text removed: "Arisutea STM32 v0.1 3x6 Design mattyams"
