File: arisutea-pcb.sch (KiCad schematic (older format))
At the start: 54 parts, among them J12 VCC, J13 D+, J14 D-, J15 GND, J16 RGB, J17 RGB_IN, J18 RGB_OUT, J2 MISO, J3 +5V, J4 SCK, J5 MOSI, J6 ~RES~, J7 GND, U1 USBLC6-2SC6, U2 ATmega32U4-AU, Y1 Crystal_GND24

Commit message: initial STM32 design
Parts:
- removed C1, C2: 22pF, arisutea:C_0805_2012Metric_Pad1.18x1.45mm_HandSolder, symbol Device:C
- removed C3: 10uF, arisutea:C_0805_2012Metric_Pad1.18x1.45mm_HandSolder, symbol Device:C
- removed C4: 1uF (±10%), arisutea:C_0805_2012Metric_Pad1.18x1.45mm_HandSolder, symbol Device:C
- removed C5: 1uF, arisutea:C_0805_2012Metric_Pad1.18x1.45mm_HandSolder, symbol Device:C
- removed C6, C7, C8, C9: 0.1uF, arisutea:C_0805_2012Metric_Pad1.18x1.45mm_HandSolder, symbol Device:C
- removed J12: VCC, arisutea:PinHeader_1x01_P2.54mm_Vertical, symbol Connector_Generic:Conn_01x01
- removed J13: D+, arisutea:PinHeader_1x01_P2.54mm_Vertical, symbol Connector_Generic:Conn_01x01
- removed J14: D-, arisutea:PinHeader_1x01_P2.54mm_Vertical, symbol Connector_Generic:Conn_01x01
- removed J15, J7: GND, arisutea:PinHeader_1x01_P2.54mm_Vertical, symbol Connector_Generic:Conn_01x01
- removed J16: RGB, arisutea:PinHeader_1x03_P2.54mm_Vertical, symbol Connector_Generic:Conn_01x03
- removed J17: RGB_IN, arisutea:PinHeader_1x03_P2.54mm_Vertical, symbol Connector_Generic:Conn_01x03
- removed J18: RGB_OUT, arisutea:PinHeader_1x03_P2.54mm_Vertical, symbol Connector_Generic:Conn_01x03
- removed J2: MISO, arisutea:PinHeader_1x01_P2.54mm_Vertical, symbol Connector_Generic:Conn_01x01
- removed J3: +5V, arisutea:PinHeader_1x01_P2.54mm_Vertical, symbol Connector_Generic:Conn_01x01
- removed J4: SCK, arisutea:PinHeader_1x01_P2.54mm_Vertical, symbol Connector_Generic:Conn_01x01
- removed J5: MOSI, arisutea:PinHeader_1x01_P2.54mm_Vertical, symbol Connector_Generic:Conn_01x01
- removed J6: ~RES~, arisutea:PinHeader_1x01_P2.54mm_Vertical, symbol Connector_Generic:Conn_01x01
- removed LED1: NUM_LOCK, arisutea:LED_IN-S124ARUW, symbol arisutea-pcb-r1:LED
- removed LED2: CAPS_LOCK, arisutea:LED_IN-S124ARUW, symbol arisutea-pcb-r1:LED
- removed LED3: FN_LED, arisutea:LED_IN-S124ARUW, symbol arisutea-pcb-r1:LED
- removed LOGO3, LOGO4: arisutea_logo, Symbol:OSHW-Logo_5.7x6mm_SilkScreen, symbol arisutea-pcb-r1:arisutea_logo
- removed LOGO5, LOGO6: arisutea_logo, arisutea:arisutea_logo, symbol arisutea-pcb-r1:arisutea_logo
- removed R1, R2: 22, arisutea:R_0805_2012Metric_Pad1.20x1.40mm_HandSolder, symbol Device:R
- removed R4: 10K, arisutea:R_0805_2012Metric_Pad1.20x1.40mm_HandSolder, symbol Device:R
- removed R7, R8, R9: 470, arisutea:R_0805_2012Metric_Pad1.20x1.40mm_HandSolder, symbol Device:R
- removed U1: USBLC6-2SC6, arisutea:SOT-23-6_Handsoldering, symbol arisutea-pcb-r1:USBLC6-2SC6-Power_Protection
- removed U2: ATmega32U4-AU, arisutea:TQFP-44_10x10mm_P0.8mm, symbol arisutea-pcb-r1:ATmega32U4-AU-MCU_Microchip_ATmega
- removed Y1: Crystal_GND24, arisutea:Crystal_SMD_TXC_7M-4Pin_3.2x2.5mm_HandSoldering, symbol Device:Crystal_GND24
- added C1: 10n, 3x6_components:C_0805_2012Metric_Pad1.18x1.45mm_HandSolder, symbol 3x6_symbols:Device_C_Small
- added C10, C4, C9: 1u, 3x6_components:C_0805_2012Metric_Pad1.18x1.45mm_HandSolder, symbol 3x6_symbols:Device_C_Small
- added C11, C12, C2, C3, C5: 100n, 3x6_components:C_0805_2012Metric_Pad1.18x1.45mm_HandSolder, symbol 3x6_symbols:Device_C_Small
- added C6, C8: 4.7u, 3x6_components:C_0805_2012Metric_Pad1.18x1.45mm_HandSolder, symbol 3x6_symbols:Device_C_Small
- added C7: 4.7n, 3x6_components:C_0805_2012Metric_Pad1.18x1.45mm_HandSolder, symbol 3x6_symbols:Device_C_Polarized_Small_US
- added D67: SMF6.0CA, 3x6_components:D_SOD-123, symbol 3x6_symbols:Device_D_TVS
- added J1: Conn_Generic_Conn_01x08, 3x6_connectors:PinHeader_2x04_P2.54mm_Vertical, symbol 3x6_symbols:Conn_Generic_Conn_01x08
- added LED1, LED2, LED3: LED, 3x6_components:LED_IN-S124ARUW, symbol 3x6_symbols:LED
- added LOGO3, LOGO4: arm_logo, 3x6_graphics:ARM_powered, symbol 3x6_symbols:LOGO
- added LOGO5, LOGO6: qmk_logo, 3x6_graphics:QMK_Logo_Light, symbol 3x6_symbols:LOGO
- added Q1: 2N7002, 3x6_components:SOT-23, symbol 3x6_symbols:2N7002
- added R1: 1M, 3x6_components:R_0805_2012Metric_Pad1.20x1.40mm_HandSolder, symbol 3x6_symbols:Device_R_Small
- added R10, R11, R9: 470, 3x6_components:R_0805_2012Metric_Pad1.20x1.40mm_HandSolder, symbol 3x6_symbols:Device_R_Small
- added R4, R8: 10K, 3x6_components:R_0805_2012Metric_Pad1.20x1.40mm_HandSolder, symbol 3x6_symbols:Device_R_Small
- added U1: STM32F072-LQFP48, 3x6_components:LQFP-48_7x7mm_P0.5mm, symbol 3x6_symbols:STM32F072-LQFP48
- added U2: TLV70233, 3x6_components:SOT-23-5_HandSoldering, symbol 3x6_symbols:TLV70233
- added U3: NUF2221W1T2G, 3x6_components:SOT-23-6_Handsoldering, symbol 3x6_symbols:NUF2221W1T2G
- F1: footprint arisutea:Fuse_1206_3216Metric_Pad1.42x1.75mm_HandSolder -> 3x6_components:Fuse_1206_3216Metric_Pad1.42x1.75mm_HandSolder; symbol Device:Polyfuse_Small -> 3x6_symbols:Device_Polyfuse_Small
- H1, H2, H3, H4, H5, H6, H7, H8: footprint arisutea:Plated_Through_Hole_M2 -> 3x6_mounting_hole:Plated_Through_Hole_M2
- LOGO1, LOGO2: symbol arisutea-pcb-r1:arisutea_logo -> 3x6_symbols:LOGO
- R2: renamed from R6; footprint arisutea:R_0805_2012Metric_Pad1.20x1.40mm_HandSolder -> 3x6_components:R_0805_2012Metric_Pad1.20x1.40mm_HandSolder; symbol Device:R -> Device:R_Small
- R3: renamed from R5; footprint arisutea:R_0805_2012Metric_Pad1.20x1.40mm_HandSolder -> 3x6_components:R_0805_2012Metric_Pad1.20x1.40mm_HandSolder; symbol Device:R -> Device:R_Small
- R7: renamed from R3; footprint arisutea:R_0805_2012Metric_Pad1.20x1.40mm_HandSolder -> 3x6_components:R_0805_2012Metric_Pad1.20x1.40mm_HandSolder; symbol Device:R -> 3x6_symbols:Device_R_Small
- SWR1: footprint arisutea:SW_SPST_TL3342 -> 3x6_components:SW_SPST_TL3342; symbol Switch:SW_Push -> 3x6_symbols:Switch_SW_Push
- USB1: footprint arisutea:USB_C_Receptacle_HRO_TYPE-C-31-M-12-HandSoldering -> 3x6_components:USB_C_Receptacle_HRO_TYPE-C-31-M-12-HandSoldering
Connections:
- net labels added: +3V3, NRST, SPI_CS, SPI_IRQ, SPI_MISO, SPI_MOSI, SPI_RES, SPI_SCK, VBUS, boot0, led1, led2, led3
- net labels removed: +5V, CAPS_L, FN_L, MISO, MOSI, NUM_L, RGB, RGB_5V, RGB_A, SCK, VCC, XTAL1, XTAL2, ~RES~
- wire segments 165 -> 209
- no-connect marks 3 -> 8
Other:
- note added: "VDDA"
- note added: "VDDIO"
- note added: "VDDIO2"
- moved on the sheet: H1, H2, H3, H4, H5, H6, H7, H8

Commit message: routing and placement work
Parts:
- added C4: 100n, 3x6_components:C_0805_2012Metric_Pad1.18x1.45mm_HandSolder, symbol 3x6_symbols:Device_C_Small
- renumbered C2 to C1, C9 to C10, C10 to C11, C11 to C12, C12 to C13, C1 to C2, C4 to C3, C6 to C5, C3 to C6, C8 to C7, C5 to C8, C7 to C9
Connections:
- net GND: now also C1.1, C2.1, C3.1, C6.1, C7.1, C8.1, D67.2 (A2), C4.1; no longer C1.2, C2.2, C3.2, C6.2, C7.2, C8.2, D67.1 (A1)
- net VBUS: now also D67.1 (A1); no longer D67.2 (A2)
- net +3V3 renamed 3.3V
- net 3.3V: now also C1.2, C2.2, C3.2, C6.2, C7.2, C8.2, C4.2; no longer C1.1, C2.1, C3.1, C6.1, C7.1, C8.1
Other:
- note removed: "VDDA"
- note removed: "VDDIO"
- note removed: "VDDIO2"
- moved on the sheet: C1, C2, C3, C5, C6, C7, C8, D67

Commit message: big update
Re-routed everything. Moved components around. Corrected gerbers and BOM/POS.  Updated library. Added renders.
Parts:
- C1, C12, C13, C4, C6, C8: footprint 3x6_components:C_0805_2012Metric_Pad1.18x1.45mm_HandSolder -> arisutea:C_0805_2012Metric_Pad1.18x1.45mm_HandSolder; symbol 3x6_symbols:Device_C_Small -> Device:C_Small; LCSC (none) -> C282732
- C10, C11, C3: footprint 3x6_components:C_0805_2012Metric_Pad1.18x1.45mm_HandSolder -> arisutea:C_0805_2012Metric_Pad1.18x1.45mm_HandSolder; symbol 3x6_symbols:Device_C_Small -> Device:C_Small; LCSC (none) -> C28323
- C2: footprint 3x6_components:C_0805_2012Metric_Pad1.18x1.45mm_HandSolder -> arisutea:C_0805_2012Metric_Pad1.18x1.45mm_HandSolder; symbol 3x6_symbols:Device_C_Small -> Device:C_Small; LCSC (none) -> C83170
- C5, C7: footprint 3x6_components:C_0805_2012Metric_Pad1.18x1.45mm_HandSolder -> arisutea:C_0805_2012Metric_Pad1.18x1.45mm_HandSolder; symbol 3x6_symbols:Device_C_Small -> Device:C_Small; LCSC (none) -> C92762
- C9: footprint 3x6_components:C_0805_2012Metric_Pad1.18x1.45mm_HandSolder -> arisutea:C_0805_2012Metric_Pad1.18x1.45mm_HandSolder; symbol 3x6_symbols:Device_C_Polarized_Small_US -> Device:C_Polarized_Small_US; LCSC (none) -> C123621
- D67: footprint 3x6_components:D_SOD-123 -> arisutea:D_SOD-123; symbol 3x6_symbols:Device_D_TVS -> Device:D_TVS; LCSC (none) -> C123791
- F1: footprint 3x6_components:Fuse_1206_3216Metric_Pad1.42x1.75mm_HandSolder -> arisutea:Fuse_1206_3216Metric_Pad1.42x1.75mm_HandSolder; LCSC (none) -> C70068
- H1, H2, H3, H4, H5, H6, H7, H8: footprint 3x6_mounting_hole:Plated_Through_Hole_M2 -> arisutea:Generic-Mounthole
- J1: footprint 3x6_connectors:PinHeader_2x04_P2.54mm_Vertical -> arisutea:PinHeader_2x04_P2.54mm_Vertical; symbol 3x6_symbols:Conn_Generic_Conn_01x08 -> Connector_Generic:Conn_01x08
- LED1, LED2, LED3: footprint 3x6_components:LED_IN-S124ARUW -> arisutea:LED_IN-S124ARUW; symbol 3x6_symbols:LED -> arisutea-pcb:LED; LCSC (none) -> C401114
- LOGO3, LOGO4: footprint 3x6_graphics:ARM_powered -> arisutea:Logo_ARM_powered; symbol 3x6_symbols:LOGO -> arisutea-pcb:LOGO
- LOGO5, LOGO6: footprint 3x6_graphics:QMK_Logo_Light -> arisutea:Logo_QMK_Light; symbol 3x6_symbols:LOGO -> arisutea-pcb:LOGO
- Q1: footprint 3x6_components:SOT-23 -> arisutea:SOT-23; symbol 3x6_symbols:2N7002 -> arisutea-pcb:2N7002; LCSC (none) -> C181082
- R1: footprint 3x6_components:R_0805_2012Metric_Pad1.20x1.40mm_HandSolder -> arisutea:R_0805_2012Metric_Pad1.20x1.40mm_HandSolder; symbol 3x6_symbols:Device_R_Small -> Device:R_Small; LCSC (none) -> C26115
- R10, R11, R4, R7, R8, R9: footprint 3x6_components:R_0805_2012Metric_Pad1.20x1.40mm_HandSolder -> arisutea:R_0805_2012Metric_Pad1.20x1.40mm_HandSolder; symbol 3x6_symbols:Device_R_Small -> Device:R_Small
- R2, R3: footprint 3x6_components:R_0805_2012Metric_Pad1.20x1.40mm_HandSolder -> arisutea:R_0805_2012Metric_Pad1.20x1.40mm_HandSolder; LCSC C27834 -> C26023
- SWR1: footprint 3x6_components:SW_SPST_TL3342 -> arisutea:SW_SPST_TL3342; symbol 3x6_symbols:Switch_SW_Push -> arisutea-pcb:Switch_SW_Push
- U1: footprint 3x6_components:LQFP-48_7x7mm_P0.5mm -> arisutea:LQFP-48_7x7mm_P0.5mm; symbol 3x6_symbols:STM32F072-LQFP48 -> arisutea-pcb:STM32F103x8_B-LQFP48; LCSC (none) -> C80488
- U2: footprint 3x6_components:SOT-23-5_HandSoldering -> arisutea:SOT-23-5_HandSoldering; symbol 3x6_symbols:TLV70233 -> arisutea-pcb:TLV70233; LCSC (none) -> C26833
- U3: footprint 3x6_components:SOT-23-6_Handsoldering -> arisutea:SOT-363_SC-70-6_Handsoldering; symbol 3x6_symbols:NUF2221W1T2G -> arisutea-pcb:NUF2221W1T2G; LCSC (none) -> C274624
- USB1: footprint 3x6_components:USB_C_Receptacle_HRO_TYPE-C-31-M-12-HandSoldering -> arisutea:USB_C_Receptacle_HRO_TYPE-C-31-M-12-HandSoldering; symbol arisutea-pcb-r1:USB_C_Receptacle_HRO_TYPE-C-31-M-12 -> arisutea-pcb:USB_C_Receptacle_HRO_TYPE-C-31-M-12; LCSC (none) -> C319148
Other:
- moved on the sheet: C1, C2, C3, C4, C5, C6, C7, C8
