File: matrix.sch (KiCad schematic (older format))
At the start: 132 parts, among them SW1 SW_Push, SW10 SW_Push, SW11 SW_Push, SW12 SW_Push, SW13 SW_Push, SW14 SW_Push, SW15 SW_Push, SW16 SW_Push, SW17 SW_Push, SW18 SW_Push, SW19 SW_Push, SW2 SW_Push, SW20 SW_Push, SW21 SW_Push, SW22 SW_Push, SW23 SW_Push, SW24 SW_Push, SW25 SW_Push, SW26 SW_Push, SW27 SW_Push, SW28 SW_Push, SW29 SW_Push, SW3 SW_Push, SW30 SW_Push, SW31 SW_Push, SW32 SW_Push, SW33 SW_Push, SW34 SW_Push, SW35 SW_Push, SW36 SW_Push, SW37 SW_Push, SW38 SW_Push, SW39 SW_Push, SW4 SW_Push, SW40 SW_Push, SW41 SW_Push, SW42 SW_Push, SW43 SW_Push, SW44 SW_Push, SW45 SW_Push, SW46 SW_Push, SW47 SW_Push, SW48 SW_Push, SW49 SW_Push, SW5 SW_Push, SW50 SW_Push, SW51 SW_Push, SW52 SW_Push, SW53 SW_Push, SW54 SW_Push, SW55 SW_Push, SW56 SW_Push, SW57 SW_Push, SW58 SW_Push, SW59 SW_Push, SW6 SW_Push, SW60 SW_Push, SW61 SW_Push, SW62 SW_Push, SW63 SW_Push, SW64 SW_Push, SW65 SW_Push, SW66 SW_Push, SW7 SW_Push, SW8 SW_Push, SW9 SW_Push

Commit message: routing and placement work
Connections:
- net row0: now also D63.1 (K)
- net row1: now also D64.1 (K); no longer D63.1 (K)
- net row2: now also D65.1 (K); no longer D64.1 (K)
- net row3: no longer D65.1 (K)
Other:
- moved on the sheet: D63, D64, D65, SW63, SW64, SW65
Changed lines of the file:
@@
 L Switch:SW_Push SW63
 U 1 1 5C66EC7D
-P 13300 4700
+P 13300 3700
 AR Path="/5C66EC7D" Ref="SW63"  Part="1"
 AR Path="/5C4EF302/5C66EC7D" Ref="SW63"  Part="1"
-F 0 "SW63" H 13300 4985 50  0000 C CNN
+F 0 "SW63" H 13300 3985 50  0000 C CNN
+F 1 "SW_Push" H 13300 3894 50  0000 C CNN
+F 2 "arisutea:SW_Hotswap_Kailh_1.00u" H 13300 3900 50  0001 C CNN
+F 3 "" H 13300 3900 50  0001 C CNN
+	1    13300 3700
+	-1   0    0    -1
+$EndComp
+$Comp
+L Device:D D63
+U 1 1 5C66EC84
+P 13500 3850
+F 0 "D63" V 13550 4050 50  0000 R CNN
+F 1 "D" V 13450 4000 50  0000 R CNN
+F 2 "arisutea:D_SOD-123" H 13500 3850 50  0001 C CNN
+F 3 "~" H 13500 3850 50  0001 C CNN
+F 4 "C81598" H 13500 3850 50  0001 C CNN "LCSC"
+	1    13500 3850
+	0    -1   -1   0
+$EndComp
+Wire Wire Line
+	13500 4000 13500 4050
+$Comp
+L Switch:SW_Push SW64
+U 1 1 5C66EC8F
+P 13300 4700
+AR Path="/5C66EC8F" Ref="SW64"  Part="1"
+AR Path="/5C4EF302/5C66EC8F" Ref="SW64"  Part="1"
+F 0 "SW64" H 13300 4985 50  0000 C CNN
 F 1 "SW_Push" H 13300 4894 50  0000 C CNN
 F 2 "arisutea:SW_Hotswap_Kailh_1.00u" H 13300 4900 50  0001 C CNN
@@
 $EndComp
 $Comp
-L Device:D D63
-U 1 1 5C66EC84
+L Device:D D64
+U 1 1 5C66ECA5
 P 13500 4850
-F 0 "D63" V 13550 5050 50  0000 R CNN
+F 0 "D64" V 13550 5050 50  0000 R CNN
 F 1 "D" V 13450 5000 50  0000 R CNN
 F 2 "arisutea:D_SOD-123" H 13500 4850 50  0001 C CNN
@@
 	0    -1   -1   0
 $EndComp
-Wire Wire Line
-	13500 5000 13500 5050
-$Comp
-L Switch:SW_Push SW64
-U 1 1 5C66EC8F
-P 13300 5750
-AR Path="/5C66EC8F" Ref="SW64"  Part="1"
-AR Path="/5C4EF302/5C66EC8F" Ref="SW64"  Part="1"
-F 0 "SW64" H 13300 6035 50  0000 C CNN
-F 1 "SW_Push" H 13300 5944 50  0000 C CNN
-F 2 "arisutea:SW_Hotswap_Kailh_1.00u" H 13300 5950 50  0001 C CNN
-F 3 "" H 13300 5950 50  0001 C CNN
-	1    13300 5750
-	-1   0    0    -1
-$EndComp
-$Comp
-L Device:D D64
-U 1 1 5C66ECA5
-P 13500 5900
-F 0 "D64" V 13550 6100 50  0000 R CNN
-F 1 "D" V 13450 6050 50  0000 R CNN
-F 2 "arisutea:D_SOD-123" H 13500 5900 50  0001 C CNN
-F 3 "~" H 13500 5900 50  0001 C CNN
-F 4 "C81598" H 13500 5900 50  0001 C CNN "LCSC"
-	1    13500 5900
-	0    -1   -1   0
-$EndComp
-Wire Wire Line
-	13500 6050 13500 6100
 Text Notes 3800 3300 0    100  ~ 0
 ESC
@@
 Text Notes 12600 4300 0    100  ~ 0
 |
-Text Notes 13250 4300 0    100  ~ 0
+Text Notes 13250 3300 0    100  ~ 0
 M1
 Connection ~ 4050 5050
@@
 Text Notes 11950 5350 0    100  ~ 0
 ENT
+Text Notes 13250 4300 0    100  ~ 0
+M2
+Wire Wire Line
+	4050 8100 5700 8100
+Wire Wire Line
+	5700 8100 7000 8100
+Wire Wire Line
+	7650 8100 8950 8100
+Wire Wire Line
+	8950 8100 10250 8100
+Wire Wire Line
+	10250 8100 12200 8100
+Wire Wire Line
+	11550 7100 12850 7100
+Wire Wire Line
+	11800 5750 11800 7750
 Text Notes 13250 5350 0    100  ~ 0
-M2
-Wire Wire Line
-	4050 8100 5700 8100
-Wire Wire Line
-	5700 8100 7000 8100
-Wire Wire Line
-	7650 8100 8950 8100
-Wire Wire Line
-	8950 8100 10250 8100
-Wire Wire Line
-	10250 8100 12200 8100
-Wire Wire Line
-	11550 7100 12850 7100
-Wire Wire Line
-	11800 5750 11800 7750
-Text Notes 13250 6350 0    100  ~ 0
 M3
 Text Notes 13250 7350 0    100  ~ 0
@@
 Connection ~ 4050 7100
 Wire Wire Line
-	13100 5750 13100 6750
-Connection ~ 13100 6750
-Wire Wire Line
-	13500 7050 13500 7100
-Wire Wire Line
 	13500 8050 13500 8100
 $Comp
@@
 L Device:D D65
 U 1 1 5C66ECAC
-P 13500 6900
-F 0 "D65" V 13550 7100 50  0000 R CNN
-F 1 "D" V 13450 7050 50  0000 R CNN
-F 2 "arisutea:D_SOD-123" H 13500 6900 50  0001 C CNN
-F 3 "~" H 13500 6900 50  0001 C CNN
-F 4 "C81598" H 13500 6900 50  0001 C CNN "LCSC"
-	1    13500 6900
+P 13500 5900
+F 0 "D65" V 13550 6100 50  0000 R CNN
+F 1 "D" V 13450 6050 50  0000 R CNN
+F 2 "arisutea:D_SOD-123" H 13500 5900 50  0001 C CNN
+F 3 "~" H 13500 5900 50  0001 C CNN
+F 4 "C81598" H 13500 5900 50  0001 C CNN "LCSC"
+	1    13500 5900
 	0    -1   -1   0
 $EndComp
@@
 	-1   0    0    -1
 $EndComp
-Wire Wire Line
-	13100 6750 13100 7750
 $Comp
 L Switch:SW_Push SW65
 U 1 1 5C66EC96
-P 13300 6750
+P 13300 5750
 AR Path="/5C66EC96" Ref="SW65"  Part="1"
 AR Path="/5C4EF302/5C66EC96" Ref="SW65"  Part="1"
-F 0 "SW65" H 13300 7035 50  0000 C CNN
-F 1 "SW_Push" H 13300 6944 50  0000 C CNN
-F 2 "arisutea:SW_Hotswap_Kailh_1.00u" H 13300 6950 50  0001 C CNN
-F 3 "" H 13300 6950 50  0001 C CNN
-	1    13300 6750
+F 0 "SW65" H 13300 6035 50  0000 C CNN
+F 1 "SW_Push" H 13300 5944 50  0000 C CNN
+F 2 "arisutea:SW_Hotswap_Kailh_1.00u" H 13300 5950 50  0001 C CNN
+F 3 "" H 13300 5950 50  0001 C CNN
+	1    13300 5750
 	-1   0    0    -1
 $EndComp
@@
 Connection ~ 12450 4700
 Connection ~ 12450 6750
-Wire Wire Line
-	13100 4700 13100 5750
-Connection ~ 13100 4700
 Connection ~ 13100 5750
 Text Notes 12500 3300 0    100  ~ 0
 BKSP
 Wire Wire Line
-	13500 5050 12850 5050
-Connection ~ 12850 5050
-Wire Wire Line
-	13500 6100 12200 6100
-Connection ~ 12200 6100
-Wire Wire Line
-	13500 7100 12850 7100
-Connection ~ 12850 7100
+	13500 4050 12850 4050
 Wire Wire Line
 	13500 8100 12850 8100
 Connection ~ 12850 8100
 Wire Wire Line
-	13100 2850 13100 4700
+	13100 2850 13100 3700
 Connection ~ 12450 3700
 Wire Wire Line
@@
 	-1   0    0    -1
 $EndComp
+Connection ~ 12850 4050
+Connection ~ 13100 3700
+Wire Wire Line
+	13100 5750 13100 7750
+Wire Wire Line
+	13100 3700 13100 4700
+Connection ~ 13100 4700
+Wire Wire Line
+	13100 4700 13100 5750
+Wire Wire Line
+	13500 5000 13500 5050
+Wire Wire Line
+	13500 5050 12850 5050
+Connection ~ 12850 5050
+Wire Wire Line
+	13500 6050 13500 6100
+Wire Wire Line
+	13500 6100 12200 6100
+Connection ~ 12200 6100
 $EndSCHEMATC
